File: Sensor_Node/Sensor_Boards/Sensor_Board_0x04_Luminosity_TSL2561_v1/Eagle/Sensor_Board_0x04_Luminosity_TSL2561_v1.sch (EAGLE design)
At the start: 16 parts, among them J1 M04_SMD_90, J2 M06_SMD_STRAIGHT, J4 ARDUINO_ISP, U2 ATMEGA328P_TQFP, Y1 8MHZ

Commit message: Changes Library & TSL2561
- moved reset path a bit around
- corrected faulty connector in library and on print
Parts:
- removed J2: M06_SMD_STRAIGHT, myownthings:M06_SMD_STRAIGHT
- added U$9: M06_SMD_STRAIGHT, wsn:M06_SMD_STRAIGHT
Connections:
- net GND: now also U$9.1; no longer J2.1
- net SCL: now also U$9.4; no longer J2.4
- net SDA: now also U$9.5; no longer J2.5
- net VCC: now also U$9.6; no longer J2.6
Changed lines of the file:
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@@
 <?xml version="1.0" encoding="utf-8"?>
 <!DOCTYPE eagle SYSTEM "eagle.dtd">
-<eagle version="8.1.1">
+<eagle version="8.2.2">
 <drawing>
 <settings>
@@
 <layer number="115" name="ReferenceISLANDS" color="7" fill="1" visible="yes" active="yes"/>
 <layer number="116" name="Patch_BOT" color="9" fill="4" visible="yes" active="yes"/>
+<layer number="117" name="BACKMAAT1" color="7" fill="1" visible="yes" active="yes"/>
 <layer number="118" name="Rect_Pads" color="7" fill="1" visible="yes" active="yes"/>
+<layer number="119" name="KAP_TEKEN" color="7" fill="1" visible="yes" active="yes"/>
+<layer number="120" name="KAP_MAAT1" color="7" fill="1" visible="yes" active="yes"/>
 <layer number="121" name="_tsilk" color="7" fill="1" visible="yes" active="yes"/>
 <layer number="122" name="_bsilk" color="7" fill="1" visible="yes" active="yes"/>
@@
 <layer number="128" name="_bValues" color="7" fill="1" visible="yes" active="yes"/>
 <layer number="129" name="Mask" color="7" fill="1" visible="yes" active="yes"/>
+<layer number="130" name="SMDSTROOK" color="7" fill="1" visible="yes" active="yes"/>
 <layer number="131" name="tAdjust" color="7" fill="1" visible="yes" active="yes"/>
 <layer number="132" name="bAdjust" color="7" fill="1" visible="yes" active="yes"/>
+<layer number="133" name="bottom_silk" color="7" fill="1" visible="yes" active="yes"/>
 <layer number="144" name="Drill_legend" color="7" fill="1" visible="yes" active="yes"/>
 <layer number="150" name="Notes" color="7" fill="1" visible="yes" active="yes"/>
@@
 <part name="U$15" library="myownthings" deviceset="N/C" device=""/>
 <part name="U$16" library="myownthings" deviceset="N/C" device=""/>
-<part name="J2" library="myownthings" deviceset="M06_SMD_STRAIGHT" device=""/>
 <part name="U$19" library="myownthings" deviceset="N/C" device=""/>
 <part name="U$20" library="myownthings" deviceset="N/C" device=""/>
@@
 <part name="P+6" library="supply1" deviceset="VCC" device=""/>
 <part name="C1" library="eagle-ltspice" deviceset="C" device="" value="100n"/>
+<part name="U$9" library="wsn" deviceset="M06_SMD_STRAIGHT" device=""/>
 </parts>
 <sheets>
@@
 <instance part="U$15" gate="G$1" x="106.68" y="93.98"/>
 <instance part="U$16" gate="G$1" x="106.68" y="91.44"/>
-<instance part="J2" gate="G$1" x="58.42" y="43.18"/>
 <instance part="U$19" gate="G$1" x="63.5" y="43.18"/>
 <instance part="U$20" gate="G$1" x="63.5" y="40.64"/>
@@
 <instance part="P+6" gate="VCC" x="134.62" y="53.34"/>
 <instance part="C1" gate="G$1" x="35.56" y="182.88" rot="R90"/>
+<instance part="U$9" gate="G$1" x="58.42" y="43.18"/>
 </instances>
 <busses>
@@
 <pinref part="GND10" gate="1" pin="GND"/>
 <wire x1="71.12" y1="38.1" x2="71.12" y2="35.56" width="0.1524" layer="91"/>
-<pinref part="J2" gate="G$1" pin="1"/>
 <wire x1="71.12" y1="38.1" x2="63.5" y2="38.1" width="0.1524" layer="91"/>
+<pinref part="U$9" gate="G$1" pin="1"/>
 </segment>
 <segment>
@@
 <pinref part="P+16" gate="VCC" pin="VCC"/>
 <wire x1="71.12" y1="50.8" x2="71.12" y2="55.88" width="0.1524" layer="91"/>
-<pinref part="J2" gate="G$1" pin="6"/>
 <wire x1="63.5" y1="50.8" x2="71.12" y2="50.8" width="0.1524" layer="91"/>
+<pinref part="U$9" gate="G$1" pin="6"/>
 </segment>
 <segment>
@@
 <wire x1="63.5" y1="45.72" x2="68.58" y2="45.72" width="0.1524" layer="91"/>
 <label x="68.58" y="45.72" size="1.27" layer="95" xref="yes"/>
-<pinref part="J2" gate="G$1" pin="4"/>
+<pinref part="U$9" gate="G$1" pin="4"/>
 </segment>
 </net>
@@
 <wire x1="63.5" y1="48.26" x2="68.58" y2="48.26" width="0.1524" layer="91"/>
 <label x="68.58" y="48.26" size="1.27" layer="95" xref="yes"/>
-<pinref part="J2" gate="G$1" pin="5"/>
-</segment>
-</net>
+<pinref part="U$9" gate="G$1" pin="5"/>
+</segment>
+</net>

Commit message: TSL2561
- reset path
- sensor connector footer
Connections:
- removed net N$4: C1.2, R5.1, S1.RIGHT, U2.PC6(/RESET)
- new net FTDI_RESET: C1.1, SV1.6
- net RESET: now also C1.2, R5.1, S1.RIGHT, U2.PC6(/RESET); no longer C1.1, SV1.6
Changed lines of the file:
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@@
 </segment>
 <segment>
-<pinref part="C1" gate="G$1" pin="1"/>
-<wire x1="33.02" y1="182.88" x2="27.94" y2="182.88" width="0.1524" layer="91"/>
-<label x="27.94" y="182.88" size="1.778" layer="95" rot="R180" xref="yes"/>
-</segment>
-<segment>
-<pinref part="SV1" gate="1" pin="6"/>
-<wire x1="116.84" y1="45.72" x2="121.92" y2="45.72" width="0.1524" layer="91"/>
-<label x="121.92" y="45.72" size="1.27" layer="95" xref="yes"/>
+<pinref part="C1" gate="G$1" pin="2"/>
+<pinref part="U2" gate="U$1" pin="PC6(/RESET)"/>
+<wire x1="40.64" y1="182.88" x2="48.26" y2="182.88" width="0.1524" layer="91"/>
+<pinref part="R5" gate="G$1" pin="1"/>
+<wire x1="48.26" y1="182.88" x2="55.88" y2="182.88" width="0.1524" layer="91"/>
+<wire x1="55.88" y1="182.88" x2="60.96" y2="182.88" width="0.1524" layer="91"/>
+<wire x1="48.26" y1="185.42" x2="48.26" y2="182.88" width="0.1524" layer="91"/>
+<junction x="48.26" y="182.88"/>
+<pinref part="S1" gate="G$1" pin="RIGHT"/>
+<wire x1="48.26" y1="180.34" x2="48.26" y2="182.88" width="0.1524" layer="91"/>
+<wire x1="55.88" y1="182.88" x2="55.88" y2="193.04" width="0.1524" layer="91"/>
+<junction x="55.88" y="182.88"/>
+<wire x1="55.88" y1="193.04" x2="68.58" y2="193.04" width="0.1524" layer="91"/>
+<label x="68.58" y="193.04" size="1.27" layer="95" xref="yes"/>
 </segment>
 </net>
@@
 <pinref part="R7" gate="G$1" pin="2"/>
 <wire x1="78.74" y1="93.98" x2="73.66" y2="93.98" width="0.1524" layer="91"/>
-<label x="73.66" y="93.98" size="1.778" layer="95" rot="R180" xref="yes"/>
+<label x="73.66" y="93.98" size="1.27" layer="95" rot="R180" xref="yes"/>
 </segment>
 </net>
@@
 <pinref part="R7" gate="G$1" pin="1"/>
 <wire x1="96.52" y1="93.98" x2="88.9" y2="93.98" width="0.1524" layer="91"/>
-</segment>
-</net>
-<net name="N$4" class="0">
-<segment>
-<pinref part="C1" gate="G$1" pin="2"/>
-<pinref part="U2" gate="U$1" pin="PC6(/RESET)"/>
-<wire x1="40.64" y1="182.88" x2="48.26" y2="182.88" width="0.1524" layer="91"/>
-<pinref part="R5" gate="G$1" pin="1"/>
-<wire x1="48.26" y1="182.88" x2="60.96" y2="182.88" width="0.1524" layer="91"/>
-<wire x1="48.26" y1="185.42" x2="48.26" y2="182.88" width="0.1524" layer="91"/>
-<junction x="48.26" y="182.88"/>
-<pinref part="S1" gate="G$1" pin="RIGHT"/>
-<wire x1="48.26" y1="180.34" x2="48.26" y2="182.88" width="0.1524" layer="91"/>
 </segment>
 </net>
@@
 </segment>
 </net>
+<net name="FTDI_RESET" class="0">
+<segment>
+<pinref part="SV1" gate="1" pin="6"/>
+<wire x1="116.84" y1="45.72" x2="121.92" y2="45.72" width="0.1524" layer="91"/>
+<label x="121.92" y="45.72" size="1.27" layer="95" xref="yes"/>
+</segment>
+<segment>
+<pinref part="C1" gate="G$1" pin="1"/>
+<wire x1="33.02" y1="182.88" x2="27.94" y2="182.88" width="0.1524" layer="91"/>
+<label x="27.94" y="182.88" size="1.27" layer="95" rot="R180" xref="yes"/>
+</segment>
+</net>

Commit message: Update SensorBoard TSL2561
new reference print - updated all placements, defined positions of
connectors and improved routing.
Parts:
- removed C10: 100n, eagle-ltspice:C
- removed U$9: M06_SMD_STRAIGHT, wsn:M06_SMD_STRAIGHT
- added C4: 100n, eagle-ltspice:C
- added SV2: (no value), con-lstb:MA06-1
- SV1: value (none) -> M06_SMD_STRAIGHT; device con-lstb:MA06-1 -> wsn:M06_SMD_STRAIGHT
- renumbered C9 to C2, R5 to R2, R7 to R1, R8 to R3, S3 to S2, U2 to U1
Connections:
- net FTDI_RESET: now also SV2.6; no longer SV1.6
- net FTDI_RXI: now also SV2.4; no longer SV1.4
- net FTDI_TXO: now also SV2.5; no longer SV1.5
- net GND: now also C4.2, SV2.1, SV2.2; no longer C10.2, SV1.2, U$9.1
- net L1: now also U1.PB2(SS/OC1B); no longer U1.PC0(ADC0)
- net N$15: now also C3.1; no longer C10.1
- net SCL: now also SV1.4; no longer U$9.4
- net SDA: now also SV1.5; no longer U$9.5
- net VCC: now also C4.1, SV1.6, SV2.3; no longer C3.1, SV1.3, U$9.6
Other:
- moved on the sheet: C3
