File: Sensor_Node/Sensor_Boards/Sensor_Board_0xXX_Protoyping/Eagle/Sensor_Board_0xXX_Prototyping_v1.brd (EAGLE design)
At the start: 55 x 35 mm, 36 parts, among them J1 M04_SMD_90, J4 ARDUINO_ISP, U2 ATMEGA328P_TQFP, Y1 8MHZ

Commit message: Updated Prototyping Board & DS18B20 Board
Parts:
- removed C10, C9: 100n, eagle-ltspice:C0805
- removed R6: 10k, SparkFun-Passives:0805
- removed R8: 330, SparkFun-Passives:0805
- added C2, C3: 100n, eagle-ltspice:C0805
- added R1: 10k, SparkFun-Passives:0805
- added R3: 330, SparkFun-Passives:0805
- moved J1 1.27 mm to (43.2, 10.2)
- moved U$2 1.27 mm to (35.6, 10.2)
- moved LED1 1.00 mm to (47.0, 24.8)
- moved U2 0.84 mm to (38.7, 18.4)
- moved S3 0.63 mm to (27.0, 21.6)
- moved SV1 0.45 mm to (52.1, 24.8)
- moved S1 0.45 mm to (23.8, 33.0)
- moved C1 0.40 mm to (36.8, 26.0)
- moved Y1 0.32 mm to (48.3, 15.2)
- moved J4 0.32 mm to (48.3, 27.9)
- renumbered R5 to R2
Connections:
- new net PC0: PAD16.1, PAD7.1, U2.23
- net DBG_ENABLE: now also R1.2; no longer R6.2
- net GND: now also C2.2, C3.2; no longer C10.2, C9.2
- net L1: now also R3.2, U2.14; no longer PAD16.1, PAD7.1, R8.2, U2.23
- net N$15: now also C3.1; no longer C10.1
- net N$3: now also R1.1; no longer R6.1
- net N$30: now also R3.1; no longer R8.1
- net VCC: now also C2.1; no longer C9.1
Routing:
- net L1: track 67.3 -> 4.78 mm, vias 3 -> 0
- net PC0: track 0.00 -> 52.2 mm, vias 0 -> 1
- net GND: track 36.5 -> 56.8 mm, vias 9 -> 7
- net VCC: track 69.9 -> 59.5 mm, vias 3 -> 2
- net FTDI_TXO: track 29.9 -> 19.5 mm, vias 2 -> 1
- net SDA: track 40.2 -> 34.1 mm, vias 2 -> 1
- net MCU_TXO: track 8.92 -> 14.9 mm
- net ADC7: track 54.6 -> 59.2 mm, vias 2 -> 1
- net N$15: track 7.95 -> 12.4 mm
- net MCU_RXI: track 20.8 -> 16.8 mm
- net MISO: track 9.74 -> 13.3 mm
- net SCK: track 11.4 -> 15.0 mm
- net PC1: track 42.0 -> 44.6 mm, vias 2 -> 1
- net PC2: track 35.3 -> 37.5 mm, vias 2 -> 1
- net +5V: track 20.1 -> 21.7 mm
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
Commit message: Finished Prototyping Board
- did some tyding up
Connections:
- net GND: now also U$1.P$1, U$1.P$2, U$1.P$3, U$1.P$4, U$1.P$5, U$1.P$6, U$1.P$7, U$1.P$8
- net INT0: now also PAD15.1, PAD6.1; no longer PAD14.1, PAD5.1
- net INT1: no longer PAD15.1, PAD6.1
- net VCC: now also PAD14.1, PAD5.1
Routing:
- net INT1: track 19.6 -> 0.00 mm, vias 2 -> 0
- net VCC: track 59.5 -> 75.4 mm
- net INT0: track 22.0 -> 20.4 mm, vias 2 -> 1
Other:
- board text added: "+3.3V"
- board text added: "D"
- board text added: "DEBUG"
- board text added: "G"
- board text added: "N"
- board text added: "RESET"
- board text removed: "INT1"
