File: Sensor_Node/Sensor_Boards/Sensor_Board_0x01_Test/Eagle/Sensor_Board_0x01_Test_v1.brd (EAGLE design)
At the start: 55 x 35 mm, 14 parts, among them J1 M04_SMD_90, J4 ARDUINO_ISP, U2 ATMEGA328P_TQFP, Y1 8MHZ

Commit message: Vorlage-Board fertig
Routing:
- net SDA: track 39.4 -> 0.00 mm, vias 2 -> 0
- net SCL: track 27.3 -> 0.00 mm, vias 2 -> 0
- net VCC: track 71.7 -> 58.1 mm
- net GND: track 64.5 -> 56.2 mm
Other:
- board text added: "A/S Vorlage-Board"
- board text removed: "A/S Sensor Board SHT31"
- board text removed: "N/C"
- board text removed: "SCL"
- board text removed: "SDA"
Changed lines of the file:
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@@
 <text x="47.625" y="11.7475" size="0.8128" layer="21">RX</text>
 <text x="49.53" y="11.7475" size="0.8128" layer="21">GND</text>
-<wire x1="1.143" y1="31.115" x2="21.463" y2="31.115" width="0.4064" layer="21"/>
-<wire x1="21.463" y1="31.115" x2="21.463" y2="20.574" width="0.4064" layer="21"/>
-<wire x1="1.143" y1="31.115" x2="1.143" y2="20.574" width="0.4064" layer="21"/>
-<wire x1="1.143" y1="20.574" x2="21.463" y2="20.574" width="0.4064" layer="21"/>
-<text x="21.1455" y="28.067" size="0.8128" layer="21" rot="R180">VCC</text>
-<text x="18.7325" y="28.067" size="0.8128" layer="21" rot="R180">GND</text>
-<text x="16.0655" y="28.067" size="0.8128" layer="21" rot="R180">SCL</text>
-<text x="13.5255" y="28.067" size="0.8128" layer="21" rot="R180">SDA</text>
-<text x="10.9855" y="28.067" size="0.8128" layer="21" rot="R180">N/C</text>
-<text x="8.4455" y="28.067" size="0.8128" layer="21" rot="R180">N/C</text>
-<text x="5.9055" y="28.067" size="0.8128" layer="21" rot="R180">N/C</text>
 <text x="3.175" y="3.175" size="1.778" layer="21">A/S
-Sensor Board SHT31</text>
+Vorlage-Board</text>
 <circle x="52.07" y="31.115" radius="1.309084375" width="0.4064" layer="21"/>
-<text x="3.4925" y="28.067" size="0.8128" layer="21" rot="R180">N/C</text>
 <text x="53.853340625" y="26.9864" size="0.8128" layer="21" rot="R270">VCC</text>
 <text x="50.68331875" y="32.9852" size="1.016" layer="21">FTDI</text>
@@
 <wire x1="23.8125" y1="33.02" x2="27.94" y2="33.02" width="0.4064" layer="1"/>
 <wire x1="27.94" y1="33.02" x2="31.7625" y2="33.02" width="0.4064" layer="1"/>
-<wire x1="17.9705" y1="33.02" x2="21.9075" y2="33.02" width="0.4064" layer="1"/>
 <wire x1="21.9075" y1="33.02" x2="23.8125" y2="33.02" width="0.4064" layer="1"/>
 <wire x1="38.335" y1="20.0025" x2="38.335" y2="19.1325" width="0.4064" layer="1"/>
@@
 <wire x1="29.845" y1="25.7175" x2="29.845" y2="24.2475" width="0.4064" layer="1"/>
 <wire x1="29.845" y1="24.2475" x2="29.6875" y2="24.09" width="0.4064" layer="1"/>
-<wire x1="20.0025" y1="26.67" x2="18.2855" y2="24.953" width="0.4064" layer="1"/>
 <wire x1="21.9075" y1="26.67" x2="28.8925" y2="26.67" width="0.4064" layer="1"/>
-<wire x1="21.9075" y1="26.67" x2="20.0025" y2="26.67" width="0.4064" layer="1"/>
-<wire x1="52.07" y1="28.575" x2="52.07" y2="31.115" width="0" layer="19" extent="1-1"/>
-<wire x1="45.94" y1="24.765" x2="52.07" y2="28.575" width="0" layer="19" extent="1-1"/>
-<wire x1="43.21" y1="30.48" x2="44.45" y2="25.0825" width="0" layer="19" extent="1-1"/>
-<wire x1="31.7625" y1="33.02" x2="35.88" y2="31.75" width="0" layer="19" extent="1-1"/>
-<wire x1="38.335" y1="22.0726" x2="44.45" y2="25.0825" width="0" layer="19" extent="1-1"/>
-<wire x1="48.26" y1="17.145" x2="45.94" y2="24.765" width="0" layer="19" extent="1-1"/>
-<wire x1="51.1175" y1="10.4775" x2="48.26" y2="15.24" width="0" layer="19" extent="1-1"/>
 </signal>
 <signal name="VCC" class="1">
@@
 <wire x1="39.6875" y1="27.305" x2="39.6875" y2="24.13" width="0.4064" layer="16"/>
 <wire x1="39.6875" y1="24.13" x2="40.005" y2="23.8125" width="0.4064" layer="16"/>
-<wire x1="16.3855" y1="13.4595" x2="18.415" y2="11.43" width="0.4064" layer="1"/>
-<wire x1="18.415" y1="11.43" x2="29.21" y2="11.43" width="0.4064" layer="1"/>
 </signal>
 <signal name="RESET">
@@
 <signal name="SCL">
 <contactref element="U2" pad="28"/>
-<via x="33.02" y="18.415" extent="1-16" drill="0.35"/>
-<wire x1="34.4424" y1="18.18" x2="33.255" y2="18.18" width="0.4064" layer="1"/>
-<wire x1="33.255" y1="18.18" x2="33.02" y2="18.415" width="0.4064" layer="1"/>
-<wire x1="33.02" y1="18.415" x2="31.115" y2="18.415" width="0.4064" layer="16"/>
-<wire x1="31.115" y1="18.415" x2="30.48" y2="17.78" width="0.4064" layer="16"/>
-<wire x1="30.48" y1="17.78" x2="18.415" y2="17.78" width="0.4064" layer="16"/>
-<wire x1="14.9225" y1="21.2725" x2="14.9225" y2="26.9875" width="0.4064" layer="16"/>
-<via x="14.9225" y="26.9875" extent="1-16" drill="0.35"/>
-<wire x1="18.415" y1="17.78" x2="14.9225" y2="21.2725" width="0.4064" layer="16"/>
-<wire x1="15.113" y1="27.178" x2="14.9225" y2="26.9875" width="0.4064" layer="1"/>
 </signal>
 <signal name="SDA">
 <contactref element="U2" pad="27"/>
-<via x="12.7" y="30.48" extent="1-16" drill="0.35"/>
-<wire x1="15.24" y1="19.3675" x2="14.9225" y2="19.685" width="0.4064" layer="16"/>
-<via x="36.195" y="18.7325" extent="1-16" drill="0.35"/>
-<wire x1="15.24" y1="19.3675" x2="17.78" y2="16.8275" width="0.4064" layer="16"/>
-<wire x1="34.29" y1="16.8275" x2="36.195" y2="18.7325" width="0.4064" layer="16"/>
-<wire x1="17.78" y1="16.8275" x2="34.29" y2="16.8275" width="0.4064" layer="16"/>
-<wire x1="12.7" y1="32.5755" x2="12.7" y2="30.48" width="0.4064" layer="1"/>
-<wire x1="12.7" y1="30.48" x2="12.7" y2="21.9075" width="0.4064" layer="16"/>
-<wire x1="12.7" y1="21.9075" x2="15.24" y2="19.3675" width="0.4064" layer="16"/>
-<wire x1="34.4424" y1="18.98" x2="35.9475" y2="18.98" width="0.4064" layer="1"/>
-<wire x1="35.9475" y1="18.98" x2="36.195" y2="18.7325" width="0.4064" layer="1"/>
 </signal>
 <signal name="L1">
