File: Sensor_Node/Sensor_Boards/Sensor_Board_0x06_CO2_S8_v2/Eagle/Sensor_Board_0x06_CO2_v2.brd (EAGLE design)
At the start: 55 x 35 mm, 24 parts, among them J1 M04_SMD_90, J4 ARDUINO_ISP, U1 CCS811, U2 ATMEGA328P_TQFP, Y1 8MHZ

Commit message: Updated CO2-Board
Parts:
- added C5: 100n, eagle-ltspice:C0805
- added JP3: (no value), SparkFun_CSS811_Breakout:SPARKFUN-JUMPERS_SMT-JUMPER_2_NO_SILK
- added R10: 10k, SparkFun-Passives:0805
- added R11: 100k, SparkFun-Passives:0805
- added U3: (no value), Adafruit SHT31 Breakout:MICROBUILDER_SHT3X
- R5, R7, R8: value 4.7k -> 10k
- moved JP1 30.9 mm to (29.5, 1.91), turned to 180 degrees
- moved R7 30.0 mm to (27.0, 5.40)
- moved R8 30.0 mm to (31.1, 5.40)
- moved R4 4.26 mm to (6.67, 20.6)
- moved R5 3.62 mm to (15.6, 29.5), turned to 0 degrees
- moved R6 3.55 mm to (6.67, 29.5)
- moved C4 2.56 mm to (15.6, 25.1)
- moved U1 2.29 mm to (11.1, 25.1)
- moved JP2 2.13 mm to (6.67, 25.1)
- moved R9 2.01 mm to (15.6, 20.6)
Connections:
- new net N$7: R10.1, U3.6
- new net N$8: JP3.2, R11.1, U3.2
- net GND: now also C5.2, JP3.1, U3.7, U3.8, U3.THERMAL
- net SCL: now also U3.4
- net SDA: now also U3.1
- net VCC: now also C5.1, R10.2, R11.2, U3.5
Routing:
- net VCC: track 58.1 -> 105.0 mm, vias 2 -> 4
- net GND: track 56.2 -> 72.9 mm, vias 6 -> 9
- net SENS_RES: track 0.00 -> 9.98 mm, vias 0 -> 2
- net N$8: track 0.00 -> 9.23 mm
- net N$4: track 0.00 -> 8.05 mm
- net NTC_SENSE: track 0.00 -> 7.69 mm
- net N$7: track 0.00 -> 7.45 mm
