File: Sensor_Node/Sensor_Boards/Sensor_Board_0x06_CO2_S8_v2/Eagle/Sensor_Board_0x06_CO2_v2.sch (EAGLE design)
At the start: 24 parts, among them J1 M04_SMD_90, J4 ARDUINO_ISP, U1 CCS811, U2 ATMEGA328P_TQFP, Y1 8MHZ

Commit message: Updated CO2-Board
Parts:
- added C5: 100n, eagle-ltspice:C
- added JP3: SPARKFUN-JUMPERS_JUMPER-SMT_2_NO_SILK, SparkFun_CSS811_Breakout:SPARKFUN-JUMPERS_JUMPER-SMT_2_NO_SILK
- added R10: 10k, SparkFun-Passives:RESISTOR0805-RES
- added R11: 100k, SparkFun-Passives:RESISTOR0805-RES
- added U3: (no value), Adafruit SHT31 Breakout:MICROBUILDER_SHT3X
- R5, R7, R8: value 4.7k -> 10k
Connections:
- new net N$7: R10.1, U3.NRESET
- new net N$8: JP3.2, R11.1, U3.ADDR
- net GND: now also C5.2, JP3.1, U3.R(VSS), U3.VSS
- net SCL: now also U3.SCL
- net SDA: now also U3.SDA
- net VCC: now also C5.1, R10.2, R11.2, U3.VDD
Other:
- note added: "JP1 connects SDA and SCL to 10k pull-up resistors."
- note removed: "JP1 connects SDA and SCL to 4.7k pull-up resistors."
- moved on the sheet: C4, JP1, R4, R7, R8, R9
