File: Sensor_Node/Sensor_Boards/Sensor_Board_0x02_Temperature_Humidity_SHT31_v2/Eagle/Sensor_Board_0x02_Temperature_Humidity_SHT31_v2.brd (EAGLE design)
At the start: 55 x 35 mm, 28 parts, among them J1 M04_SMD_90, J4 ARDUINO_ISP, U1 CCS811, U2 ATMEGA328P_TQFP, Y1 8MHZ

Commit message: Version 2 of CO2 and SHT31 - Sensorboards
Parts:
- removed C5: 100n, eagle-ltspice:C0805
- removed JP2: (no value), SparkFun_CSS811_Breakout:SPARKFUN-JUMPERS_SMT-JUMPER_2_NO_SILK
- removed R10, R7, R8, R9: 10k, SparkFun-Passives:0805
- removed R11, R6: 100k, SparkFun-Passives:0805
- removed U3: (no value), Adafruit SHT31 Breakout:MICROBUILDER_SHT3X
- R4: device SparkFun_CSS811_Breakout:CCS811_BREAKOUT_TEMP_0603 -> SparkFun-Passives:0805
- R5: value 10k -> 100k
- U1: value CCS811 -> (none); device SparkFun_CSS811_Breakout:CCS811_BREAKOUT_TEMP_LGA10 -> Adafruit SHT31 Breakout:MICROBUILDER_SHT3X
- moved R5 10.1 mm to (6.03, 26.7)
- moved R4 6.98 mm to (6.03, 29.5), turned to 0 degrees
- moved JP1 4.97 mm to (10.5, 24.8), turned to 180 degrees
- moved U1 1.59 mm to (10.5, 28.6), turned to 90 degrees
- moved C4 0.45 mm to (15.2, 26.7), turned to 180 degrees
Connections:
- removed net AUX: R4.1, R9.1, U1.8
- removed net N$7: R10.1, U3.6
- removed net N$8: JP2.2, R11.1, U3.2
- removed net NTC_SENSE: R4.2, U1.4, U1.5
- removed net SENS_RES: R5.1, U1.2
- removed net SENS_WAKE: U1.7
- new net N$5: JP1.2, R5.1, U1.2
- net GND: now also U1.7, U1.8, U1.THERMAL; no longer C5.2, JP2.1, U1.EP, U3.7, U3.8, U3.THERMAL
- net N$4: now also R4.1, U1.6; no longer JP1.2, R6.1, U1.1
- net SCL: now also U1.4; no longer R8.1, U1.10, U3.4
- net SDA: now also U1.1; no longer R7.1, U1.9, U3.1
- net VCC: now also R4.2, U1.5; no longer C5.1, R10.2, R11.2, R6.2, R7.2, R8.2, R9.2, U1.6, U3.5
Routing:
- net SDA: track 79.3 -> 35.8 mm, vias 4 -> 2
- net VCC: track 130.0 -> 102.9 mm
- net SCL: track 53.6 -> 32.1 mm, vias 6 -> 2
- net AUX: track 12.7 -> 0.00 mm, vias 2 -> 0
- net SENS_RES: track 9.98 -> 0.00 mm, vias 2 -> 0
- net GND: track 78.8 -> 69.2 mm, vias 9 -> 7
- net N$5: track 0.00 -> 9.23 mm
- net N$8: track 9.23 -> 0.00 mm
- net NTC_SENSE: track 7.70 -> 0.00 mm
- net N$7: track 7.45 -> 0.00 mm
- net N$4: track 8.05 -> 7.45 mm
Other:
- board text added: "A/S Vorlage-Board"
- board text removed: "A/S Sensor Board CO2"
- board text removed: "CCS811"
