File: Miscellaneous/Eagle/SensorBoards_Combined_Mask_20_01_2018.brd (EAGLE design)
At the start: 143 parts, among them J1 M04_SMD_90, J10 1x3 RA Female .1", J11 ARDUINO_ISP, J12 M04_SMD_90, J2 ARDUINO_ISP, J3 M04_SMD_90, J4 ARDUINO_ISP, J5 ARDUINO_ISP, J6 M04_SMD_90, J7 5.5x2.1mm Barrel, J8 ARDUINO_ISP, J9 1x3 RA Female .1", U10 ATMEGA328P_TQFP, U2 ATMEGA328P_TQFP, U3 ATMEGA328P_TQFP, U4 MIKE-TEMP_TSL2561FN, U5 ATMEGA328P_TQFP, U6 ATMEGA328P_TQFP, U7 CCS811, U9 ATMEGA328P_TQFP, Y1 8MHZ, Y2 8MHZ, Y3 8MHZ, Y4 8MHZ, Y5 8MHZ, Y6 8MHZ

Commit message: Various changes
- updated two masks
- changed combined mask again
- tiedied up CO2 sensor a bit
- used another footprint for TSL2561-sensor
Parts:
- added R36: 10k, SparkFun-Passives:0805
- J5: value ARDUINO_ISP -> 5.5x2.1mm Barrel; device marc_library:M-2X3 -> wsn:POWER_JACK_SMD
- J6: value M04_SMD_90 -> ARDUINO_ISP; device myownthings:M04_SMD_90 -> marc_library:M-2X3
- J7: value 5.5x2.1mm Barrel -> M04_SMD_90; device wsn:POWER_JACK_SMD -> myownthings:M04_SMD_90
- JP2: device TSL2561 Luminosity Sensor BOB:MIKE-TEMP_SJ_3 -> SparkFun_CSS811_Breakout:SPARKFUN-JUMPERS_SMT-JUMPER_2_NO_SILK
- JP4: device SparkFun_CSS811_Breakout:SPARKFUN-JUMPERS_SMT-JUMPER_2_NO_SILK -> TSL2561 Luminosity Sensor BOB:MIKE-TEMP_SJ_3
- R11, R21: value 10k -> 100k
- R19: value 330 -> 10k
- R20: device SparkFun_CSS811_Breakout:CCS811_BREAKOUT_TEMP_0603 -> SparkFun-Passives:0805
- R25: value 10k -> 330
- R27: value 100k -> 10k
- R9: device SparkFun-Passives:0805 -> SparkFun_CSS811_Breakout:CCS811_BREAKOUT_TEMP_0603
- U4: value MIKE-TEMP_TSL2561FN -> CCS811; device TSL2561 Luminosity Sensor BOB:MIKE-TEMP_FN-6 -> SparkFun_CSS811_Breakout:CCS811_BREAKOUT_TEMP_LGA10
- U6: value ATMEGA328P_TQFP -> (none); device marc_library:TQFP32-08 -> Adafruit SHT31 Breakout:MICROBUILDER_SHT3X
- U7: value CCS811 -> ATMEGA328P_TQFP; device SparkFun_CSS811_Breakout:CCS811_BREAKOUT_TEMP_LGA10 -> marc_library:TQFP32-08
- U8: value (none) -> MIKE-TEMP_TSL2561T; device Adafruit SHT31 Breakout:MICROBUILDER_SHT3X -> TSL2561 Luminosity Sensor BOB:MIKE-TEMP_TMB-6
- moved C8 66.9 mm to (74.0, 67.9), turned to 180 degrees
- moved C17 65.8 mm to (7.62, 59.4), turned to 0 degrees
- moved R23 64.0 mm to (31.4, 51.8)
- moved R24 63.6 mm to (25.1, 51.8)
- moved JP4 62.5 mm to (6.67, 63.5), turned to 270 degrees
- moved R10 60.8 mm to (73.0, 70.8), turned to 0 degrees
- moved U4 57.8 mm to (68.6, 66.0)
- moved U8 57.7 mm to (11.1, 63.5), turned to 0 degrees
- moved JP2 57.5 mm to (64.1, 66.0), turned to 90 degrees
- moved R11 56.6 mm to (64.1, 70.5)
- moved C14 56.0 mm to (38.1, 69.8)
- moved C15 56.0 mm to (38.1, 66.7)
- moved R7 55.9 mm to (81.0, 51.8)
- moved S2 55.9 mm to (81.0, 71.1)
- moved S7 55.9 mm to (25.1, 71.1)
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Connections:
- removed net SENS_WAKE: U7.7
- new net N$39: JP4.2, U8.2
- net AUX: now also R19.1, R9.1, U4.8; no longer R20.1, R25.1, U7.8
- net DBG_ENABLE3: now also R24.2, U7.26; no longer R18.2, U6.26
- net FTDI_RESET3: now also C16.1; no longer C15.1
- net FTDI_RXI3: now also U7.30; no longer U6.30
- net FTDI_TXO3: now also U7.31; no longer U6.31
- net GND1: now also C13.2, C8.2, J5.GND, J5.P$4, JP2.1, JP3.1, R22.1, U4.EP, U6.7, U6.8, U6.THERMAL; no longer C8.1, JP2.3, U4.3
- net GND3: now also C15.2, C17.1, J6.P$5, J7.4, JP4.3, U7.21, U7.3, U7.5, U8.3; no longer C13.2, C16.2, C17.2, J5.P$5, J6.4, J7.GND, J7.P$4, JP3.1, JP4.1, U6.21, U6.3, U6.5, U7.EP, U8.7, U8.8, U8.THERMAL
- net L4: now also R25.2, U7.14; no longer R19.2, U6.14
- net MCU_RXI3: now also J7.3, U7.11; no longer J6.3, U6.11
- net MCU_TXO3: now also J7.2, U7.10; no longer J6.2, U6.10
- net MISO3: now also J6.P$1, U7.16; no longer J5.P$1, U6.16
- net MOSI3: now also J6.P$3, U7.15; no longer J5.P$3, U6.15
- net N$11: now also JP2.2, U4.1; no longer JP2.1
- net N$12: now also R20.1, U6.6; no longer JP2.2, U4.2
- net N$20: now also JP3.2, R21.1, U6.2; no longer U6.8, Y4.3
- net N$21: now also R22.2, U4.7; no longer U6.7, Y4.1
- net N$22: now also U7.8, Y4.3; no longer LED4.A, R19.1
- net N$23: now also U7.7, Y4.1; no longer C13.1, U6.20
- net N$24: now also LED4.A, R25.1; no longer R18.1, S8.2
- net N$25: now also C14.1, U7.20; no longer JP3.2, R22.1, U7.1
- net N$26: now also R24.1, S8.2; no longer R26.1, U8.6
- net N$27: now also JP4.1, R36.1; no longer JP4.2, R27.1, U8.2
- net NTC_SENSE: now also R9.2, U4.4, U4.5; no longer R20.2, U7.4, U7.5
- net RESET3: now also C16.2, J6.P$4, R23.1, U7.29; no longer C15.2, J5.P$4, R17.1, U6.29
- net SCK3: now also J6.P$2, U7.17; no longer J5.P$2, U6.17
- net SCL1: now also R18.1, U4.10, U6.4; no longer R9.1, U4.4
- net SCL2: now also R26.1, U7.28; no longer R24.1, U6.28, U7.10
- net SDA1: now also R17.1, U4.9, U6.1; no longer R10.1, U4.6
- net SDA2: now also R27.1, U7.27, U8.6; no longer R23.1, U6.27, U7.9, U8.1
- net SENS_RES: now also R10.1, U4.2; no longer R21.1, U7.2
- net VCC1: now also C13.1, C8.1, J5.VIN0, J5.VIN1, R17.2, R18.2, R19.2, R20.2, R21.2, U4.6, U6.5; no longer C8.2, R9.2, U4.1
- net VCC3: now also C15.1, C17.2, J6.P$6, J7.1, R36.2, U7.18, U7.4, U8.1; no longer C14.1, C16.1, C17.1, J5.P$6, J6.1, J7.VIN0, J7.VIN1, R17.2, R21.2, R22.2, R24.2, R25.2, U6.18, U6.4, U6.6, U8.5
