File: Sensor_Node/Sensor_Boards/Previous Versions/Sensor_Board_0x07_Heat_Flux_v1/Eagle/Sensor_Board_0x07_Heat_Flux.sch (EAGLE design)
At the start: 24 parts, among them IC1 MCP3911A0-E/SS, IC2 4066D, U1 PIC16F1825-I/ST-TSSOP14, X1 22-23-2041

Commit message: Work on heat flux sensor continued
Parts:
- IC1: SPICEPREFIX (none) -> X
