File: Sensor_Node/Sensor_modules/Sensor_Module_0x02_Temperature_Humidity_SHT31_v2/Eagle/Sensor_Module_0x02_Temperature_Humidity_SHT31_v2.brd (EAGLE design)
At the start: 55 x 35 mm, 19 parts, among them J1 M04_SMD_90, J4 ARDUINO_ISP, U2 ATMEGA328P_TQFP, Y1 8MHZ

Commit message: Renaming boards to modules inside eagle files
Other:
- board text added: "A/S Sensor Module - SHT31 v2"
- board text removed: "A/S Sensor Board - SHT31"
Changed lines of the file:
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@@
 <?xml version="1.0" encoding="utf-8"?>
 <!DOCTYPE eagle SYSTEM "eagle.dtd">
-<eagle version="8.5.1">
+<eagle version="9.1.1">
 <drawing>
 <settings>
@@
 <text x="49.53" y="11.7475" size="0.8128" layer="21">GND</text>
 <text x="3.175" y="3.175" size="1.778" layer="21">A/S
-Sensor Board - SHT31</text>
+Sensor Module - SHT31 v2</text>
 <circle x="52.07" y="31.115" radius="1.309084375" width="0.4064" layer="21"/>
 <text x="53.853340625" y="26.9864" size="0.8128" layer="21" rot="R270">VCC</text>
@@
 <param name="checkStop" value="0"/>
 <param name="checkValues" value="0"/>
+<param name="checkNames" value="1"/>
+<param name="checkWireStubs" value="1"/>
+<param name="checkPolygonWidth" value="0"/>
 <param name="useDiameter" value="13"/>
 <param name="maxErrors" value="50"/>
@@
 </signal>
 </signals>
+<mfgpreviewcolors>
+<mfgpreviewcolor name="soldermaskcolor" color="0xC8008000"/>
+<mfgpreviewcolor name="silkscreencolor" color="0xFFFEFEFE"/>
+<mfgpreviewcolor name="backgroundcolor" color="0xFF282828"/>
+<mfgpreviewcolor name="coppercolor" color="0xFFFFBF00"/>
+<mfgpreviewcolor name="substratecolor" color="0xFF786E46"/>
+</mfgpreviewcolors>
 </board>
 </drawing>
