File: Sensor_Node/Sensor_modules/Sensor_Module_0x05_0x09_0x10_0x11_Pulse_v1/Eagle/Sensor_Module_0x09_0x10_Pulse_v1.sch (EAGLE design)
At the start: 21 parts, among them U2 ATMEGA328P_TQFP, Y1 8MHZ

Commit message: Renaming boards to modules inside eagle files
Other:
- note added: "Interrupt connector to Main Module"
- note added: "Main Module Connector"
- note added: "Sensor Module - Pulse v1"
- note removed: "Communication Module Connector"
- note removed: "Interrupt to CommBoard"
- note removed: "Sensor Board - Pulse"
Changed lines of the file:
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@@
 <?xml version="1.0" encoding="utf-8"?>
 <!DOCTYPE eagle SYSTEM "eagle.dtd">
-<eagle version="8.4.1">
+<eagle version="9.1.1">
 <drawing>
 <settings>
@@
 <wire x1="48.26" y1="43.18" x2="48.26" y2="12.7" width="0.1524" layer="97" style="shortdash"/>
 <wire x1="48.26" y1="12.7" x2="7.62" y2="12.7" width="0.1524" layer="97" style="shortdash"/>
-<text x="10.16" y="38.1" size="1.778" layer="97">Communication Module Connector</text>
+<text x="10.16" y="38.1" size="1.778" layer="97">Main Module Connector</text>
 <wire x1="144.78" y1="66.04" x2="53.34" y2="66.04" width="0.1524" layer="97" style="shortdash"/>
 <wire x1="53.34" y1="12.7" x2="53.34" y2="66.04" width="0.1524" layer="97" style="shortdash"/>
@@
 <wire x1="53.34" y1="114.3" x2="53.34" y2="68.58" width="0.1524" layer="97" style="shortdash"/>
 <text x="55.88" y="111.125" size="1.778" layer="97">Digital Input 2</text>
-<text x="10.16" y="73.025" size="1.778" layer="97">Interrupt to CommBoard</text>
+<text x="10.16" y="73.025" size="1.778" layer="97">Interrupt connector to Main Module</text>
 <text x="99.06" y="99.06" size="1.778" layer="97">PULL UP/DOWN
 only connect one</text>
 <text x="278.4475" y="1.27" size="2.54" layer="94" font="vector">1.0</text>
-<text x="224.4725" y="11.1125" size="2.54" layer="94" font="vector">Sensor Board - Pulse</text>
+<text x="224.4725" y="11.1125" size="2.54" layer="94" font="vector">Sensor Module - Pulse v1</text>
 <wire x1="149.86" y1="58.42" x2="195.58" y2="58.42" width="0.1524" layer="97" style="shortdash"/>
 <wire x1="195.58" y1="58.42" x2="195.58" y2="12.7" width="0.1524" layer="97" style="shortdash"/>
