File: Sensor_Node/Sensor_modules/Sensor_Module_0x08_Dual_Temperatures_2xDS18B20_v1/Eagle/Sensor_Module_0x08_Dual_Temperatures_2xDS18B20_v1.brd (EAGLE design)
At the start: 55 x 35 mm, 18 parts, among them J2 1x3 RA Female .1", J3 1x3 RA Female .1", J4 ARDUINO_ISP, U2 ATMEGA328P_TQFP, Y1 8MHZ

Commit message: Renaming boards to modules inside eagle files
Other:
- board text added: "A/S Sensor Module - 2xDS18B20 v1"
- board text removed: "A/S Sensor Board - 2xDS18B20"
Changed lines of the file:
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@@
 <?xml version="1.0" encoding="utf-8"?>
 <!DOCTYPE eagle SYSTEM "eagle.dtd">
-<eagle version="8.4.3">
+<eagle version="9.1.1">
 <drawing>
 <settings>
@@
 <text x="17.78" y="23.8125" size="0.8128" layer="21">GND</text>
 <text x="3.175" y="3.175" size="1.778" layer="21">A/S
-Sensor Board - 2xDS18B20</text>
+Sensor Module - 2xDS18B20 v1</text>
 <hole x="19.3675" y="29.845" drill="2.54"/>
 <hole x="9.68375" y="29.845" drill="2.54"/>
@@
 <param name="checkRestrict" value="1"/>
 <param name="checkStop" value="0"/>
+<param name="checkValues" value="0"/>
+<param name="checkNames" value="1"/>
+<param name="checkWireStubs" value="1"/>
+<param name="checkPolygonWidth" value="0"/>
 <param name="useDiameter" value="13"/>
 <param name="maxErrors" value="50"/>
@@
 </signal>
 </signals>
+<mfgpreviewcolors>
+<mfgpreviewcolor name="soldermaskcolor" color="0xC8008000"/>
+<mfgpreviewcolor name="silkscreencolor" color="0xFFFEFEFE"/>
+<mfgpreviewcolor name="backgroundcolor" color="0xFF282828"/>
+<mfgpreviewcolor name="coppercolor" color="0xFFFFBF00"/>
+<mfgpreviewcolor name="substratecolor" color="0xFF786E46"/>
+</mfgpreviewcolors>
 </board>
 </drawing>
