File: Sensor_Node/Sensor_modules/Sensor_Module_0x12_U-Value/Eagle/Sensor_Module_0x12_U-Value_v1.brd (EAGLE design)
At the start: 55 x 35 mm, 42 parts, among them IC1 MCP3911, IC2 40XX_4066D, IC4 MAX31855, J1 M04_SMD_90, J4 ARDUINO_ISP, U2 ATMEGA328P_TQFP, Y1 8MHZ

Commit message: Renaming boards to modules inside eagle files
Other:
- board text added: "A/S Sensor Module U-Value v1"
- board text removed: "A/S Sensor Board Heat Flux"
Changed lines of the file:
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@@
 <?xml version="1.0" encoding="utf-8"?>
 <!DOCTYPE eagle SYSTEM "eagle.dtd">
-<eagle version="8.7.0">
+<eagle version="9.1.1">
 <drawing>
 <settings>
@@
 <text x="49.53" y="11.7475" size="0.8128" layer="21">GND</text>
 <text x="2.06375" y="1.5875" size="1.4224" layer="21">A/S
-Sensor Board
-Heat Flux</text>
+Sensor Module
+U-Value v1</text>
 <circle x="52.07" y="31.115" radius="1.309084375" width="0.4064" layer="21"/>
 <text x="53.853340625" y="26.9864" size="0.8128" layer="21" rot="R270">VCC</text>
@@
 <param name="checkStop" value="0"/>
 <param name="checkValues" value="0"/>
+<param name="checkNames" value="1"/>
+<param name="checkWireStubs" value="1"/>
+<param name="checkPolygonWidth" value="0"/>
 <param name="useDiameter" value="13"/>
 <param name="maxErrors" value="50"/>
@@
 </signal>
 </signals>
+<mfgpreviewcolors>
+<mfgpreviewcolor name="soldermaskcolor" color="0xC8008000"/>
+<mfgpreviewcolor name="silkscreencolor" color="0xFFFEFEFE"/>
+<mfgpreviewcolor name="backgroundcolor" color="0xFF282828"/>
+<mfgpreviewcolor name="coppercolor" color="0xFFFFBF00"/>
+<mfgpreviewcolor name="substratecolor" color="0xFF786E46"/>
+</mfgpreviewcolors>
 </board>
 </drawing>
