File: Sensor_Node/Sensor_modules/Sensor_Module_0x12_U-Value/Eagle/Sensor_Module_0x12_U-Value_v1.sch (EAGLE design)
At the start: 42 parts, among them IC1 MCP3911, IC2 40XX_4066D, IC4 MAX31855, J1 M04_SMD_90, J4 ARDUINO_ISP, U2 ATMEGA328P_TQFP, Y1 8MHZ

Commit message: Renaming boards to modules inside eagle files
Other:
- note added: "Main Module Connector"
- note added: "Sensor Module - U-Value v1"
- note removed: "Communication Module Connector"
- note removed: "Sensor Board - MCP3911"
Changed lines of the file:
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@@
 <?xml version="1.0" encoding="utf-8"?>
 <!DOCTYPE eagle SYSTEM "eagle.dtd">
-<eagle version="8.7.0">
+<eagle version="9.1.1">
 <drawing>
 <settings>
@@
 <wire x1="47.752" y1="63.246" x2="47.752" y2="30.226" width="0.1524" layer="97" style="shortdash"/>
 <wire x1="47.752" y1="30.226" x2="7.62" y2="30.226" width="0.1524" layer="97" style="shortdash"/>
-<text x="8.89" y="60.071" size="1.778" layer="97">Communication Module Connector</text>
-<text x="224.527240625" y="11.421534375" size="2.54" layer="94" font="vector">Sensor Board - MCP3911</text>
+<text x="8.89" y="60.071" size="1.778" layer="97">Main Module Connector</text>
+<text x="224.527240625" y="11.421534375" size="2.54" layer="94" font="vector">Sensor Module - U-Value v1</text>
 <text x="277.8550125" y="1.158059375" size="2.54" layer="94" font="vector">2.0</text>
 <wire x1="109.22" y1="63.5" x2="58.42" y2="63.5" width="0.1524" layer="97" style="shortdash"/>
